File: PCB/Simon-Big-Keyboard-V2.kicad_pcb (KiCad board)
At the start: 2 copper layers, 353.5 x 125 mm, 177 parts, among them SW1 SW_Push, SW10 SW_Push, SW11 SW_Push, SW12 SW_Push, SW13 SW_Push, SW14 SW_Push, SW15 SW_Push, SW16 SW_Push, SW17 SW_Push, SW18 SW_Push, SW19 SW_Push, SW2 SW_Push, SW20 SW_Push, SW21 SW_Push, SW22 SW_Push, SW23 SW_Push, SW24 SW_Push, SW25 SW_Push, SW26 SW_Push, SW27 SW_Push, SW28 SW_Push, SW29 SW_Push, SW3 SW_Push, SW30 SW_Push, SW31 SW_Push, SW32 SW_Push, SW33 SW_Push, SW34 SW_Push, SW35 SW_Push, SW36 SW_Push, SW37 SW_Push, SW38 SW_Push, SW39 SW_Push, SW4 SW_Push, SW40 SW_Push, SW41 SW_Push, SW42 SW_Push, SW43 SW_Push, SW44 SW_Push, SW45 SW_Push, SW46 SW_Push, SW47 SW_Push, SW48 SW_Push, SW49 SW_Push, SW5 SW_Push, SW50 SW_Push, SW51 SW_Push, SW52 SW_Push, SW53 SW_Push, SW54 SW_Push, SW55 SW_Push, SW56 SW_Push, SW57 SW_Push, SW58 SW_Push, SW59 SW_Push, SW6 SW_Push, SW60 SW_Push, SW61 SW_Push, SW62 SW_Push, SW63 SW_Push, SW64 SW_Push, SW65 SW_Push, SW66 SW_Push, SW67 SW_Push, SW68 SW_Push, SW69 SW_Push, SW7 SW_Push, SW70 SW_Push, SW71 SW_Push, SW72 SW_Push, SW73 SW_Push, SW74 SW_Push, SW75 SW_Push, SW76 SW_Push, SW77 SW_Push, SW78 SW_Push, SW79 SW_Push, SW8 SW_Push, SW80 SW_Push, SW81 SW_Push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

Commit message: Add files via upload
Parts:
- A1: footprint Module:RaspberryPi_Pico_W_SMD_HandSolder -> Module:RaspberryPi_Pico_Common_THT
- SW30: footprint Button_Switch_Keyboard:SW_Cherry_MX_1.00u_PCB -> Button_Switch_Keyboard:SW_Cherry_MX_2.00u_PCB
- SW34: footprint Button_Switch_Keyboard:SW_Cherry_MX_1.00u_PCB -> Button_Switch_Keyboard:SW_Cherry_MX_1.50u_Plate
- SW47: footprint Button_Switch_Keyboard:SW_Cherry_MX_1.00u_PCB -> Button_Switch_Keyboard:SW_Cherry_MX_1.50u_PCB
- SW51: footprint Button_Switch_Keyboard:SW_Cherry_MX_1.00u_PCB -> Button_Switch_Keyboard:SW_Cherry_MX_1.75u_PCB
- SW63, SW64: footprint Button_Switch_Keyboard:SW_Cherry_MX_1.00u_PCB -> Button_Switch_Keyboard:SW_Cherry_MX_2.25u_PCB
- SW75: footprint Button_Switch_Keyboard:SW_Cherry_MX_1.00u_PCB -> Button_Switch_Keyboard:SW_Cherry_MX_2.75u_PCB
- SW77, SW78, SW79, SW81, SW82, SW83, SW84: footprint Button_Switch_Keyboard:SW_Cherry_MX_1.00u_PCB -> Button_Switch_Keyboard:SW_Cherry_MX_1.25u_PCB
- SW80: footprint Button_Switch_Keyboard:SW_Cherry_MX_1.00u_PCB -> Button_Switch_Keyboard:SW_Cherry_MX_6.25u_PCB
- moved A1 25.6 mm to (338.5, 62.4), turned to -90 degrees
- moved REF** 12.1 mm to (280.1, 90.7)
- moved D75 5.41 mm to (245.2, 82.7)
- moved D78 5.35 mm to (14.7, 100.2)
- moved D84 4.45 mm to (264.1, 101.8)
- moved D77 2.70 mm to (2.65, 99.5)
- moved D46 2.70 mm to (237.9, 41.2)
- moved D83 1.95 mm to (241.9, 100.5)
- moved D65 1.86 mm to (21.6, 80.0)
- moved D64 1.01 mm to (0.90, 80.5)
Connections:
- A1 pad 1: unconnected-(A1-GPIO0-Pad1) -> /col17
- A1 pad 11: /col6 -> /col12
- A1 pad 12: /col5 -> /col13
- A1 pad 14: /col4 -> /row0
- A1 pad 15: /col3 -> /col14
- A1 pad 16: /col2 -> unconnected-(A1-GPIO12-Pad16)
- A1 pad 17: /col1 -> unconnected-(A1-GPIO13-Pad17)
- A1 pad 19: /col0 -> /row2
- A1 pad 2: /col16 -> /col0
- A1 pad 21: /row0 -> /col15
- A1 pad 22: /row1 -> /row3
- A1 pad 24: /row2 -> /col11
- A1 pad 25: unconnected-(A1-GPIO19-Pad25) -> /col10
- A1 pad 26: /col12 -> /col9
- A1 pad 27: /col13 -> /col8
- A1 pad 29: /col17 -> /col7
- A1 pad 31: /row3 -> /col6
- A1 pad 32: /col14 -> /col5
- A1 pad 34: /col15 -> /col16
- A1 pad 4: /col11 -> /col1
- A1 pad 5: /col10 -> /col2
- A1 pad 6: /col9 -> /col3
- A1 pad 7: /col8 -> /col4
- A1 pad 9: /col7 -> /row1
Routing:
- net /col12: track 516.1 -> 325.3 mm, vias 0 -> 2
- net /col16: track 341.0 -> 154.0 mm, vias 0 -> 2
- net Net-(A1-GND-Pad13): track 221.1 -> 95.9 mm, vias 0 -> 4
- net /row3: track 382.7 -> 326.1 mm
- net /col15: track 185.5 -> 133.2 mm
- net /col1: track 430.5 -> 458.3 mm
- net /col9: track 349.3 -> 322.9 mm
- net /col0: track 467.7 -> 493.4 mm
- net /col2: track 448.8 -> 473.6 mm
- net /col3: track 439.7 -> 462.8 mm
- net /row5: track 357.2 -> 378.3 mm, vias 0 -> 1
- net /col4: track 422.5 -> 443.4 mm
- net /col8: track 357.7 -> 338.7 mm
- net /row4: track 308.0 -> 326.6 mm
- net /col7: track 376.4 -> 366.6 mm
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Other:
- board size 353.5 x 125 mm -> 353.5 x 125.7 mm

Commit message: Add files via upload
Parts:
- removed A1: RaspberryPi_Pico_W, Module:RaspberryPi_Pico_Common_THT
- added A2: RaspberryPi_Pico, Module:RaspberryPi_Pico_SMD_HandSolder, B.Cu at (314.8, 72.1)
Routing:
- net GND: track 0.00 -> 112.1 mm
- net Net-(A1-GND-Pad13): track 95.9 -> 0.00 mm, vias 4 -> 0
- net /col6: track 346.7 -> 372.2 mm, vias 0 -> 1
- net /col3: track 462.8 -> 438.3 mm, vias 0 -> 1
- net /col2: track 473.6 -> 449.2 mm, vias 0 -> 1
- net /col4: track 443.4 -> 419.4 mm, vias 0 -> 1
- net /col1: track 458.3 -> 435.7 mm, vias 0 -> 1
- net /col0: track 493.4 -> 471.3 mm, vias 0 -> 1
- net /col14: track 275.2 -> 295.1 mm, vias 0 -> 1
- net /col12: track 325.3 -> 345.2 mm, vias 2 -> 3
- net /row1: track 376.6 -> 396.1 mm, vias 0 -> 1
- net /row0: track 399.6 -> 419.1 mm, vias 1 -> 2
- net /col13: track 334.1 -> 353.6 mm, vias 0 -> 1
- net /row4: track 326.6 -> 307.1 mm
- net /row2: track 344.1 -> 363.6 mm, vias 0 -> 1
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