File: PCB/Simon-Big-Keyboard-V2.kicad_sch (KiCad schematic)
At the start: 175 parts, among them SW1 SW_Push, SW10 SW_Push, SW11 SW_Push, SW12 SW_Push, SW13 SW_Push, SW14 SW_Push, SW15 SW_Push, SW16 SW_Push, SW17 SW_Push, SW18 SW_Push, SW19 SW_Push, SW2 SW_Push, SW20 SW_Push, SW21 SW_Push, SW22 SW_Push, SW23 SW_Push, SW24 SW_Push, SW25 SW_Push, SW26 SW_Push, SW27 SW_Push, SW28 SW_Push, SW29 SW_Push, SW3 SW_Push, SW30 SW_Push, SW31 SW_Push, SW32 SW_Push, SW33 SW_Push, SW34 SW_Push, SW35 SW_Push, SW36 SW_Push, SW37 SW_Push, SW38 SW_Push, SW39 SW_Push, SW4 SW_Push, SW40 SW_Push, SW41 SW_Push, SW42 SW_Push, SW43 SW_Push, SW44 SW_Push, SW45 SW_Push, SW46 SW_Push, SW47 SW_Push, SW48 SW_Push, SW49 SW_Push, SW5 SW_Push, SW50 SW_Push, SW51 SW_Push, SW52 SW_Push, SW53 SW_Push, SW54 SW_Push, SW55 SW_Push, SW56 SW_Push, SW57 SW_Push, SW58 SW_Push, SW59 SW_Push, SW6 SW_Push, SW60 SW_Push, SW61 SW_Push, SW62 SW_Push, SW63 SW_Push, SW64 SW_Push, SW65 SW_Push, SW66 SW_Push, SW67 SW_Push, SW68 SW_Push, SW69 SW_Push, SW7 SW_Push, SW70 SW_Push, SW71 SW_Push, SW72 SW_Push, SW73 SW_Push, SW74 SW_Push, SW75 SW_Push, SW76 SW_Push, SW77 SW_Push, SW78 SW_Push, SW79 SW_Push, SW8 SW_Push, SW80 SW_Push, SW81 SW_Push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

Commit message: Add files via upload
Parts:
- A1: footprint Module:RaspberryPi_Pico_W_SMD_HandSolder -> Module:RaspberryPi_Pico_Common_THT; JLCPCB Part # (none) -> C7203002
- D1, D10, D11, D12, D13, D14, D15, D16, D17, D18, D19, D2, D20, D21, D22, D23, D24, D25, D26, D27, D28, D29, D3, D30, D31, D32, D33, D34, D35, D36, D37, D38, D39, D4, D40, D41, D42, D43, D44, D45, D46, D47, D48, D49, D5, D50, D51, D52, D53, D54, D55, D56, D57, D58, D59, D6, D60, D61, D62, D63, D64, D65, D66, D67, D68, D69, D7, D70, D71, D72, D73, D74, D75, D76, D77, D78, D79, D8, D80, D81, D82, D83, D84, D85, D86, D87, D9: JLCPCB Part # (none) -> C81598
- SW30: footprint Button_Switch_Keyboard:SW_Cherry_MX_1.00u_PCB -> Button_Switch_Keyboard:SW_Cherry_MX_2.00u_PCB
- SW34: footprint Button_Switch_Keyboard:SW_Cherry_MX_1.00u_PCB -> Button_Switch_Keyboard:SW_Cherry_MX_1.50u_Plate
- SW47: footprint Button_Switch_Keyboard:SW_Cherry_MX_1.00u_PCB -> Button_Switch_Keyboard:SW_Cherry_MX_1.50u_PCB
- SW51: footprint Button_Switch_Keyboard:SW_Cherry_MX_1.00u_PCB -> Button_Switch_Keyboard:SW_Cherry_MX_1.75u_PCB
- SW63, SW64: footprint Button_Switch_Keyboard:SW_Cherry_MX_1.00u_PCB -> Button_Switch_Keyboard:SW_Cherry_MX_2.25u_PCB
- SW75: footprint Button_Switch_Keyboard:SW_Cherry_MX_1.00u_PCB -> Button_Switch_Keyboard:SW_Cherry_MX_2.75u_PCB
- SW77, SW78, SW79, SW81, SW82, SW83, SW84: footprint Button_Switch_Keyboard:SW_Cherry_MX_1.00u_PCB -> Button_Switch_Keyboard:SW_Cherry_MX_1.25u_PCB
- SW80: footprint Button_Switch_Keyboard:SW_Cherry_MX_1.00u_PCB -> Button_Switch_Keyboard:SW_Cherry_MX_6.25u_PCB
Connections:
- net col0: now also A1.2 (GPIO1); no longer A1.19 (GPIO14)
- net col1: now also A1.4 (GPIO2); no longer A1.17 (GPIO13)
- net col10: now also A1.25 (GPIO19); no longer A1.5 (GPIO3)
- net col11: now also A1.24 (GPIO18); no longer A1.4 (GPIO2)
- net col12: now also A1.11 (GPIO8); no longer A1.26 (GPIO20)
- net col13: now also A1.12 (GPIO9); no longer A1.27 (GPIO21)
- net col14: now also A1.15 (GPIO11); no longer A1.32 (GPIO27_ADC1)
- net col15: now also A1.21 (GPIO16); no longer A1.34 (GPIO28_ADC2)
- net col16: now also A1.34 (GPIO28_ADC2); no longer A1.2 (GPIO1)
- net col17: now also A1.1 (GPIO0); no longer A1.29 (GPIO22)
- net col2: now also A1.5 (GPIO3); no longer A1.16 (GPIO12)
- net col3: now also A1.6 (GPIO4); no longer A1.15 (GPIO11)
- net col4: now also A1.7 (GPIO5); no longer A1.14 (GPIO10)
- net col5: now also A1.32 (GPIO27_ADC1); no longer A1.12 (GPIO9)
- net col6: now also A1.31 (GPIO26_ADC0); no longer A1.11 (GPIO8)
- net col7: now also A1.29 (GPIO22); no longer A1.9 (GPIO6)
- net col8: now also A1.27 (GPIO21); no longer A1.7 (GPIO5)
- net col9: now also A1.26 (GPIO20); no longer A1.6 (GPIO4)
- net row0: now also A1.14 (GPIO10); no longer A1.21 (GPIO16)
- net row1: now also A1.9 (GPIO6); no longer A1.22 (GPIO17)
- net row2: now also A1.19 (GPIO14); no longer A1.24 (GPIO18)
- net row3: now also A1.22 (GPIO17); no longer A1.31 (GPIO26_ADC0)

Commit message: Add files via upload
Parts:
- removed A1: RaspberryPi_Pico_W, Module:RaspberryPi_Pico_Common_THT, symbol MCU_Module:RaspberryPi_Pico_W
- added A2: RaspberryPi_Pico, Module:RaspberryPi_Pico_SMD_HandSolder, symbol MCU_Module:RaspberryPi_Pico
Connections:
- net col0: now also A2.2 (GPIO1)
- net col1: now also A2.4 (GPIO2)
- net col10: now also A2.25 (GPIO19)
- net col11: now also A2.24 (GPIO18)
- net col12: now also A2.11 (GPIO8)
- net col13: now also A2.12 (GPIO9)
- net col14: now also A2.15 (GPIO11)
- net col15: now also A2.21 (GPIO16)
- net col16: now also A2.34 (GPIO28_ADC2)
- net col17: now also A2.1 (GPIO0)
- net col2: now also A2.5 (GPIO3)
- net col3: now also A2.6 (GPIO4)
- net col4: now also A2.7 (GPIO5)
- net col5: now also A2.32 (GPIO27_ADC1)
- net col6: now also A2.31 (GPIO26_ADC0)
- net col7: now also A2.29 (GPIO22)
- net col8: now also A2.27 (GPIO21)
- net col9: now also A2.26 (GPIO20)
- net row0: now also A2.14 (GPIO10)
- net row1: now also A2.9 (GPIO6)
- net row2: now also A2.19 (GPIO14)
- net row3: now also A2.22 (GPIO17)
- net row4: now also A2.10 (GPIO7)
- net row5: now also A2.20 (GPIO15)
- new net GND: A2.13 (GND), A2.18 (GND), A2.23 (GND), A2.28 (GND), A2.3 (GND), A2.38 (GND), A2.8 (GND)
- no-connect marks 0 -> 7
Changed lines of the file:
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@@
 		(color 0 0 0 0)
 	)
+	(no_connect
+		(at 68.58 82.55)
+	)
+	(no_connect
+		(at 68.58 67.31)
+	)
+	(no_connect
+		(at 50.8 21.59)
+	)
+	(no_connect
+		(at 45.72 21.59)
+	)
+	(no_connect
+		(at 40.64 21.59)
+	)
+	(no_connect
+		(at 22.86 39.37)
+	)
+	(no_connect
+		(at 22.86 36.83)
+	)
 	(wire
 		(pts
@@
 	)
 	(symbol
+		(lib_id "MCU_Module:RaspberryPi_Pico")
+		(at 45.72 59.69 0)
+		(unit 1)
+		(body_style 1)
+		(exclude_from_sim no)
+		(in_bom yes)
+		(on_board yes)
+		(in_pos_files yes)
+		(dnp no)
+		(fields_autoplaced yes)
+		(property "Reference" "A2"
+			(at 47.8633 93.98 0)
+			(show_name no)
+			(do_not_autoplace no)
+			(effects
+				(font
+					(size 1.27 1.27)
+				)
+				(justify left)
+			)
+		)
+		(property "Value" "RaspberryPi_Pico"
+			(at 47.8633 96.52 0)
+			(show_name no)
+			(do_not_autoplace no)
+			(effects
+				(font
+					(size 1.27 1.27)
+				)
+				(justify left)
+			)
+		)
+		(property "Footprint" "Module:RaspberryPi_Pico_SMD_HandSolder"
+			(at 45.72 106.68 0)
+			(hide yes)
+			(show_name no)
+			(do_not_autoplace no)
+			(effects
+				(font
+					(size 1.27 1.27)
+				)
+			)
+		)
+		(property "Datasheet" "https://datasheets.raspberrypi.com/pico/pico-datasheet.pdf"
+			(at 45.72 109.22 0)
+			(hide yes)
+			(show_name no)
+			(do_not_autoplace no)
+			(effects
+				(font
+					(size 1.27 1.27)
+				)
+			)
+		)
+		(property "Description" "Versatile and inexpensive microcontroller module powered by RP2040 dual-core Arm Cortex-M0+ processor up to 133 MHz, 264kB SRAM, 2MB QSPI flash; also supports Raspberry Pi Pico 2"
+			(at 45.72 111.76 0)
+			(hide yes)
+			(show_name no)
+			(do_not_autoplace no)
+			(effects
+				(font
+					(size 1.27 1.27)
+				)
+			)
+		)
+		(pin "2"
+		)
+		(pin "4"
+		)
+		(pin "1"
+		)
+		(pin "3"
+		)
+		(pin "15"
+		)
+		(pin "6"
+		)
+		(pin "28"
+		)
+		(pin "12"
+		)
+		(pin "14"
+		)
+		(pin "16"
+		)
+		(pin "7"
+		)
+		(pin "8"
+		)
+		(pin "13"
+		)
+		(pin "17"
+		)
+		(pin "19"
+		)
+		(pin "22"
+		)
+		(pin "23"
+		)
+		(pin "11"
+		)
+		(pin "24"
+		)
+		(pin "25"
+		)
+		(pin "34"
+		)
+		(pin "21"
+		)
+		(pin "5"
+		)
+		(pin "18"
+		)
+		(pin "20"
+		)
+		(pin "26"
+		)
+		(pin "9"
+		)
+		(pin "10"
+		)
+		(pin "27"
+		)
+		(pin "29"
+		)
+		(pin "30"
+		)
+		(pin "32"
+		)
+		(pin "33"
+		)
+		(pin "35"
+		)
+		(pin "36"
+		)
+		(pin "31"
+		)
+		(pin "37"
+		)
+		(pin "38"
+		)
+		(pin "39"
+		)
+		(pin "40"
+		)
+		(instances
+			(project "Simon-Big-Keyboard-V2"
+				(path "/1f15bbb2-91c3-480d-819a-c7e448aae989"
+					(reference "A2")
+					(unit 1)
+				)
+			)
+		)
+	)
+	(symbol
 		(lib_id "Switch:SW_Push")
 		(at 354.33 99.06 0)
@@
 	)
 	(symbol
-		(lib_id "MCU_Module:RaspberryPi_Pico_W")
-		(at 45.72 59.69 0)
-		(unit 1)
-		(body_style 1)
-		(exclude_from_sim no)
-		(in_bom yes)
-		(on_board yes)
-		(in_pos_files yes)
-		(dnp no)
-		(fields_autoplaced yes)
-		(property "Reference" "A1"
-			(at 47.8633 93.98 0)
-			(show_name no)
-			(do_not_autoplace no)
-			(effects
-				(font
-					(size 1.27 1.27)
-				)
-				(justify left)
-			)
-		)
-		(property "Value" "RaspberryPi_Pico_W"
-			(at 47.8633 96.52 0)
-			(show_name no)
-			(do_not_autoplace no)
-			(effects
-				(font
-					(size 1.27 1.27)
-				)
-				(justify left)
-			)
-		)
-		(property "Footprint" "Module:RaspberryPi_Pico_Common_THT"
-			(at 45.72 106.68 0)
-			(hide yes)
-			(show_name no)
-			(do_not_autoplace no)
-			(effects
-				(font
-					(size 1.27 1.27)
-				)
-			)
-		)
-		(property "Datasheet" "https://datasheets.raspberrypi.com/picow/pico-w-datasheet.pdf"
-			(at 45.72 109.22 0)
-			(hide yes)
-			(show_name no)
-			(do_not_autoplace no)
-			(effects
-				(font
-					(size 1.27 1.27)
-				)
-			)
-		)
-		(property "Description" "Versatile and inexpensive wireless microcontroller module powered by RP2040 dual-core Arm Cortex-M0+ processor up to 133 MHz, 264kB SRAM, 2MB QSPI flash, Infineon CYW43439 2.4GHz 802.11n wireless LAN; also supports Raspberry Pi Pico 2 W"
-			(at 45.72 111.76 0)
-			(hide yes)
-			(show_name no)
-			(do_not_autoplace no)
-			(effects
-				(font
-					(size 1.27 1.27)
-				)
-			)
-		)
-		(property "JLCPCB Part #" "C7203002"
-			(at 45.72 59.69 0)
-			(hide yes)
-			(show_name no)
-			(do_not_autoplace no)
-			(effects
-				(font
-					(size 1.27 1.27)
-				)
-			)
-		)
-		(pin "3"
-		)
-		(pin "4"
-		)
-		(pin "1"
-		)
-		(pin "2"
-		)
-		(pin "9"
-		)
-		(pin "24"
-		)
-		(pin "21"
-		)
-		(pin "27"
-		)
-		(pin "31"
-		)
-		(pin "15"
-		)
-		(pin "18"
-		)
-		(pin "17"
-		)
-		(pin "20"
-		)
-		(pin "26"
-		)
-		(pin "28"
-		)
-		(pin "23"
-		)
-		(pin "40"
-		)
-		(pin "11"
-		)
-		(pin "7"
-		)
-		(pin "8"
-		)
-		(pin "6"
-		)
-		(pin "5"
-		)
-		(pin "10"
-		)
-		(pin "12"
-		)
-		(pin "13"
-		)
-		(pin "14"
-		)
-		(pin "16"
-		)
-		(pin "19"
-		)
-		(pin "22"
-		)
-		(pin "25"
-		)
-		(pin "29"
-		)
-		(pin "30"
-		)
-		(pin "32"
-		)
-		(pin "34"
-		)
-		(pin "35"
-		)
-		(pin "36"
-		)
-		(pin "37"
-		)
-		(pin "38"
-		)
-		(pin "39"
-		)
-		(pin "33"
-		)
-		(instances
-			(project "Simon-Big-Keyboard-V2"
-				(path "/1f15bbb2-91c3-480d-819a-c7e448aae989"
-					(reference "A1")
-					(unit 1)
-				)
-			)
-		)
-	)
-	(symbol
 		(lib_id "Device:D")
 		(at 177.8 78.74 180)
@@
 					(unit 1)
 				)
+			)
+		)
+	)
+	(symbol
+		(lib_id "power:GND")
+		(at 45.72 95.25 0)
+		(unit 1)
+		(body_style 1)
+		(exclude_from_sim no)
+		(in_bom yes)
+		(on_board yes)
+		(in_pos_files yes)
+		(dnp no)
+		(fields_autoplaced yes)
+		(property "Reference" "#PWR01"
+			(at 45.72 101.6 0)
+			(hide yes)
+			(show_name no)
+			(do_not_autoplace no)
+			(effects
+				(font
+					(size 1.27 1.27)
+				)
+			)
+		)
+		(property "Value" "GND"
+			(at 45.72 100.33 0)
+			(show_name no)
+			(do_not_autoplace no)
+			(effects
+				(font
+					(size 1.27 1.27)
+				)
+			)
+		)
+		(property "Footprint" ""
+			(at 45.72 95.25 0)
+			(hide yes)
+			(show_name no)
+			(do_not_autoplace no)
+			(effects
+				(font
+					(size 1.27 1.27)
+				)
+			)
+		)
+		(property "Datasheet" ""
+			(at 45.72 95.25 0)
+			(hide yes)
+			(show_name no)
+			(do_not_autoplace no)
+			(effects
+				(font
+					(size 1.27 1.27)
+				)
+			)
+		)
+		(property "Description" "Power symbol creates a global label with name \"GND\" , ground"
+			(at 45.72 95.25 0)
+			(hide yes)
+			(show_name no)
+			(do_not_autoplace no)
+			(effects
+				(font
+					(size 1.27 1.27)
+				)
+			)
+		)
+		(pin "1"
+		)
+		(instances
+			(project "Simon-Big-Keyboard-V2"
+				(path "/1f15bbb2-91c3-480d-819a-c7e448aae989"
+					(reference "#PWR01")
+					(unit 1)
+				)
